File: kicad/esp32_spot_welder.kicad_pcb (KiCad board)
At the start: 2 copper layers, 9 parts, among them J1 Conn_01x02_Female, J2 LCD_PINS, J3 ROT_ENCD, J4 SWITCH, K1 RAYEX-L90BS, Q1 BC547, U1 L7805, U2 ESP32-DEVKITC-32D

Commit message: kicad changed
Parts:
- removed K1: RAYEX-L90BS, modules:Relay_1-Form-A_Schrack-RYII_RM5mm
- removed Q1: BC547, Package_TO_SOT_THT:TO-92_Inline
- removed R1: R, Resistor_THT:R_Axial_DIN0207_L6.3mm_D2.5mm_P10.16mm_Horizontal
- added J5: SSR_CON, TerminalBlock_Philmore:TerminalBlock_Philmore_TB132_1x02_P5.00mm_Horizontal, F.Cu at (145.6, 135.6)
- J4: footprint Connector_PinHeader_1.00mm:PinHeader_1x02_P1.00mm_Vertical -> TerminalBlock_Philmore:TerminalBlock_Philmore_TB132_1x02_P5.00mm_Horizontal
Connections:
- U2 pad 27: Net-(R1-Pad2) -> SSR_IN
Routing:
- net +12V: track 88.5 -> 5.19 mm
- net Net-(K1-PadA2): track 26.3 -> 0.00 mm
- net GND: track 112.0 -> 87.6 mm
- net Net-(R1-Pad2): track 14.9 -> 0.00 mm
- net Net-(Q1-Pad2): track 6.35 -> 0.00 mm

Commit message: updated kicad
Parts:
- removed J1: Conn_01x02_Female, Connector_PinHeader_1.00mm:PinHeader_1x02_P1.00mm_Vertical
- removed U1: L7805, Package_TO_SOT_THT:TO-220-3_Vertical
- added J6: POWER, TerminalBlock_Philmore:TerminalBlock_Philmore_TB132_1x02_P5.00mm_Horizontal, F.Cu at (88.4, 137.0)
- J2: footprint Connector_PinHeader_1.00mm:PinHeader_1x04_P1.00mm_Vertical -> Connector_PinHeader_2.00mm:PinHeader_1x04_P2.00mm_Vertical
- J3: footprint Connector_PinHeader_1.00mm:PinHeader_1x05_P1.00mm_Vertical -> Connector_PinHeader_2.00mm:PinHeader_1x05_P2.00mm_Vertical
- moved J5 22.3 mm to (132.2, 117.8), turned to 270 degrees
- moved J4 19.1 mm to (132.2, 132.0), turned to 270 degrees
- moved J3 2.20 mm to (91.6, 116.2)
Routing:
- net SW: track 8.46 -> 30.0 mm
- net SSR_IN: track 0.00 -> 13.3 mm
- net GND: track 87.6 -> 100.6 mm
- net LCD_SDA: track 46.0 -> 58.0 mm
- net +12V: track 5.19 -> 0.00 mm
- net ENC_CLK: track 6.45 -> 5.02 mm
- net +5V: track 43.0 -> 44.1 mm
- net +3V3: track 24.5 -> 25.4 mm
- net LCD_SCL: track 44.6 -> 43.9 mm
